File: hardware/sx1280_tranceiver.kicad_sch (KiCad schematic)
At the start: 15 parts, among them J1 Conn_02x06_Odd_Even, U1 sx1280, U2 2450FM07D0034, Y1 ECS-520-12-37B-CTN-TR

Commit message: finalized schematic
Parts:
- removed AE1: Antenna_Shield, Connector_Coaxial:U.FL_Hirose_U.FL-R-SMT-1_Vertical, symbol Device:Antenna_Shield
- added C10, C9: ~, Capacitor_SMD:C_0402_1005Metric, symbol Device:C_Small
- added J2: U.FL-R-SMT-1(80), Connector_Coaxial:U.FL_Hirose_U.FL-R-SMT-1_Vertical, symbol Connector:Conn_Coaxial
- added L1, L2: 0R, Inductor_SMD:L_0402_1005Metric, symbol Device:L_Small
- added R2, R3: 0R, Resistor_SMD:R_0402_1005Metric, symbol Device:R_Small
- AE3: value Antenna_Chip -> 2450AT18A100E; footprint (none) -> RF_Antenna:Johanson_2450AT18x100; LCSC (none) -> C89334
- C1: value 470n -> 470n / 50V; LCSC (none) -> C6684936; Mouser (none) -> 81-GRM155R61H474ME1D
- C2, C3: value 6p -> 6p / 50V; LCSC (none) -> C1575
- C4: Mouser (none) -> 81-GRM155R6YA105ME1J
- C5, C7, C8: Mouser (none) -> 810-C1005X6S1H104KBB
- C6: value 10n -> 10n / 50V; LCSC (none) -> C60133
- R1: value 0 -> 0R
- U1: LCSC (none) -> C125969; Mouser (none) -> 947-SX1280IMLTRT
- U2: LCSC (none) -> C2651081
- Y1: LCSC (none) -> C781783; Mouser (none) -> 520-520-12-37B-CTNTR
Connections:
- net GND: now also C10.2, C9.2, J2.2 (Ext)
- net at U2.3 (OUT): now also R2.2, R3.2
- net at AE3.1 (FEED): now also C10.1, L2.2
- new net: C9.1, J2.1 (In), L1.2
- new net ANT_CHIP: L2.1, R3.1
- new net ANT_SMA: L1.1, R2.1
- no-connect marks 1 -> 2
Other:
- note added: "0R to select desired antenna."
- note added: "optional matching circuit, place 0R in place of L if not used."
- moved on the sheet: AE3, C1, C6, C8, U1, U2
