File: hardware/sx1280_tranceiver.kicad_sch (KiCad schematic)
At the start: 21 parts, among them J1 Conn_02x06_Odd_Even, J2 U.FL-R-SMT-1(80), U1 sx1280, U2 2450FM07D0034, Y1 ECS-520-12-37B-CTN-TR

Commit message: layout
Parts:
- added L3: 15u, Inductor_SMD:L_0805_2012Metric, symbol Device:L_Small
- renumbered AE3 to AE1, C4 to C1, C1 to C2, C5 to C3, C8 to C4, C7 to C5, C2 to C7, C3 to C8, J2 to J1, J1 to J2
Connections:
- net GND: now also Y1.2, Y1.4
- net VDD_IN: now also L3.1
- net at U1.14 (DCC_SW): now also L3.2
- net ANT_SW: no longer names the net of J2.12 (Pin_12)
- no-connect marks 2 -> 1
Other:
- moved on the sheet: AE1, C10, C2, C4, C6, C9, J1, L1, L2, R2, R3, U1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

Commit message: finalized layout, added part numbers
Parts:
- AE1: Mouser (none) -> 609-2450AT18A100E
- J1: LCSC (none) -> C88374; Mouser (none) -> 798-UFLRSMT180
- U2: Mouser (none) -> 609-2450FM07A0029T
Changed lines of the file:
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@@
       (effects (font (size 1.27 1.27)) hide)
     )
-    (property "Datasheet" " ~" (at 175.26 104.14 0)
+    (property "Datasheet" "https://datasheet.lcsc.com/lcsc/1811091710_HRS-Hirose-U-FL-R-SMT-1-80_C88374.pdf" (at 175.26 104.14 0)
+      (effects (font (size 1.27 1.27)) hide)
+    )
+    (property "LCSC" "C88374" (at 175.26 104.14 0)
+      (effects (font (size 1.27 1.27)) hide)
+    )
+    (property "Mouser" " 798-UFLRSMT180 " (at 175.26 104.14 0)
       (effects (font (size 1.27 1.27)) hide)
     )
@@
       (effects (font (size 1.27 1.27)) hide)
     )
+    (property "Mouser" " 609-2450FM07A0029T " (at 90.17 124.46 0)
+      (effects (font (size 1.27 1.27)) hide)
+    )
     (pin "1")
     (pin "2")
@@
       (effects (font (size 1.27 1.27)) hide)
     )
+    (property "Mouser" " 609-2450AT18A100E " (at 176.53 135.89 0)
+      (effects (font (size 1.27 1.27)) hide)
+    )

Commit message: added part numbers for bom
Parts:
- L1, L2, R2, R3: Mouser (none) -> 71-RCA04020000ZSED
- R1: LCSC (none) -> C17168; Mouser (none) -> 71-RCA04020000ZSED
Changed lines of the file:
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@@
       (effects (font (size 1.27 1.27)) hide)
     )
-    (property "Mouser" "" (at 111.76 124.46 0)
+    (property "Mouser" " 71-RCA04020000ZSED " (at 111.76 124.46 0)
       (effects (font (size 1.27 1.27)) hide)
     )
@@
       (effects (font (size 1.27 1.27)) hide)
     )
+    (property "Mouser" " 71-RCA04020000ZSED " (at 147.32 104.14 0)
+      (effects (font (size 1.27 1.27)) hide)
+    )
     (pin "1")
     (pin "2")
@@
       (effects (font (size 1.27 1.27)) hide)
     )
+    (property "LCSC" "C17168" (at 64.77 31.75 0)
+      (effects (font (size 1.27 1.27)) hide)
+    )
+    (property "Mouser" " 71-RCA04020000ZSED " (at 64.77 31.75 0)
+      (effects (font (size 1.27 1.27)) hide)
+    )
     (pin "1")
     (pin "2")
@@
     )
     (property "Datasheet" "~" (at 147.32 139.7 0)
+      (effects (font (size 1.27 1.27)) hide)
+    )
+    (property "Mouser" " 71-RCA04020000ZSED " (at 147.32 139.7 0)
       (effects (font (size 1.27 1.27)) hide)
     )
@@
       (effects (font (size 1.27 1.27)) hide)
     )
-    (property "Mouser" "" (at 111.76 139.7 0)
-      (effects (font (size 1.27 1.27)) hide)
-    )
+    (property "Mouser" " 71-RCA04020000ZSED " (at 111.76 139.7 0)
+      (effects (font (size 1.27 1.27)) hide)
+    )
